File: ESP12E BOB_1.sch (KiCad schematic (older format))
At the start: 20 parts, among them M1 ESP-12E, P1 CONN_01X07, P2 CONN_01X13, P3 CONN_01X13, P4 CONN_01X01, P5 CONN_01X01, P6 CONN_01X01, P7 CONN_01X01, Q1 BSS138, Q2 BSS138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

Commit message: ADDED FILES
Parts:
- removed P1: CONN_01X07, symbol CONN_01X07
- added P8: CONN_01X07, symbol CONN_01X07
Connections:
- net +3V3: now also M1.8 (VCC), P3.10 (P10)
- net +5V: now also P8.3 (P3)
- net DTR: now also P8.7 (P7)
- net GND: now also P8.1 (P1)
- net RX: now also M1.21 (RXD0), P2.4 (P4), P8.4 (P4); no longer M1.22 (TXD0), P2.3 (P3)
- net TX: now also M1.22 (TXD0), P2.3 (P3), P8.5 (P5); no longer M1.21 (RXD0), P2.4 (P4)
- no-connect marks 2 -> 6
Other:
- moved on the sheet: P6
Changed lines of the file:
@@
 	5650 4150 5650 4550
 Wire Wire Line
-	5750 4150 5750 4550
+	5750 4150 5750 4950
 Wire Wire Line
 	4740 4020 4740 4190
@@
 	4650 4440 4850 4440
 Wire Wire Line
-	4850 4440 4850 4550
+	4850 4440 4850 4950
 Wire Wire Line
 	4950 2200 4950 2390
@@
 79 E3 73 01 AA 0D CF 9F 3C 98 C5 F6 CF AC 04 72 85 62 D7 80 77 B1 8B CB 18 6F AC E9 6A 17 BB B8
 C2 B0 6B C0 BB D8 C5 65 8C 5D 03 DE C5 2E 2E 63 EC 1A F0 2E 76 71 19 63 D7 80 77 B1 8B CB 18 BB
-06 BC 8B 5D 5C C6 F8 FF 01 52 B3 1C 8C A4 9D 25 1B 00 00 00 00 49 45 4E 44 AE 42 60 82 15
+06 BC 8B 5D 5C C6 F8 FF 01 52 B3 1C 8C A4 9D 25 1B 00 00 00 00 49 45 4E 44 AE 42 60 82 DA
 EndData
 $EndBitmap
-Text Label 5150 2350 1    60   ~ 0
+Text Label 5050 2700 1    60   ~ 0
 TX
-Text Label 5050 2350 1    60   ~ 0
+Text Label 5150 2700 1    60   ~ 0
 RX
 Text Label 4350 4350 0    60   ~ 0
@@
 	0    -1   1    0
 $EndComp
-$Comp
-L CONN_01X07 P1
-U 1 1 556CEEA3
-P 2600 1900
-F 0 "P1" H 2600 2300 50  0000 C CNN
-F 1 "CONN_01X07" V 2700 1900 50  0000 C CNN
-F 2 "" H 2600 1900 60  0000 C CNN
-F 3 "" H 2600 1900 60  0000 C CNN
-	1    2600 1900
-	1    0    0    -1
-$EndComp
-Text Label 2400 1700 2    60   ~ 0
-DTR
-Text Label 2400 1900 2    60   ~ 0
-RX
-Text Label 2400 2000 2    60   ~ 0
-TX
-$Comp
-L +5V #PWR018
-U 1 1 556CF6A4
-P 2400 2200
-F 0 "#PWR018" H 2400 2050 60  0001 C CNN
-F 1 "+5V" V 2400 2400 60  0000 C CNN
-F 2 "" H 2400 2200 60  0000 C CNN
-F 3 "" H 2400 2200 60  0000 C CNN
-	1    2400 2200
-	0    -1   -1   0
-$EndComp
-$Comp
-L GND #PWR019
-U 1 1 556CF802
-P 1950 2100
-F 0 "#PWR019" H 1950 1850 60  0001 C CNN
-F 1 "GND" H 1950 1950 60  0000 C CNN
-F 2 "" H 1950 2100 60  0000 C CNN
-F 3 "" H 1950 2100 60  0000 C CNN
-	1    1950 2100
-	0    1    1    0
-$EndComp
-Wire Wire Line
-	1950 2100 2400 2100
-NoConn ~ 2400 1600
-NoConn ~ 2400 1800
 Wire Wire Line
 	6050 2200 6050 2330
@@
 L CONN_01X01 P4
 U 1 1 5576BDB1
-P 8110 1760
-F 0 "P4" H 8110 1860 50  0000 C CNN
-F 1 "CONN_01X01" V 8210 1760 50  0000 C CNN
-F 2 "" H 8110 1760 60  0000 C CNN
-F 3 "" H 8110 1760 60  0000 C CNN
-	1    8110 1760
+P 8100 1750
+F 0 "P4" H 8100 1850 50  0000 C CNN
+F 1 "CONN_01X01" V 8200 1750 50  0000 C CNN
+F 2 "" H 8100 1750 60  0000 C CNN
+F 3 "" H 8100 1750 60  0000 C CNN
+	1    8100 1750
 	0    1    1    0
 $EndComp
@@
 L CONN_01X01 P5
 U 1 1 5576BFB1
-P 8690 1760
-F 0 "P5" H 8690 1860 50  0000 C CNN
-F 1 "CONN_01X01" V 8790 1760 50  0000 C CNN
-F 2 "" H 8690 1760 60  0000 C CNN
-F 3 "" H 8690 1760 60  0000 C CNN
-	1    8690 1760
+P 8700 1750
+F 0 "P5" H 8700 1850 50  0000 C CNN
+F 1 "CONN_01X01" V 8800 1750 50  0000 C CNN
+F 2 "" H 8700 1750 60  0000 C CNN
+F 3 "" H 8700 1750 60  0000 C CNN
+	1    8700 1750
 	0    1    1    0
 $EndComp
@@
 L CONN_01X01 P6
 U 1 1 5576C098
-P 9220 1760
-F 0 "P6" H 9220 1860 50  0000 C CNN
-F 1 "CONN_01X01" V 9320 1760 50  0000 C CNN
-F 2 "" H 9220 1760 60  0000 C CNN
-F 3 "" H 9220 1760 60  0000 C CNN
-	1    9220 1760
+P 9200 1750
+F 0 "P6" H 9200 1850 50  0000 C CNN
+F 1 "CONN_01X01" V 9300 1750 50  0000 C CNN
+F 2 "" H 9200 1750 60  0000 C CNN
+F 3 "" H 9200 1750 60  0000 C CNN
+	1    9200 1750
 	0    1    1    0
 $EndComp
@@
 L CONN_01X01 P7
 U 1 1 5576C13E
-P 9800 1760
-F 0 "P7" H 9800 1860 50  0000 C CNN
-F 1 "CONN_01X01" V 9900 1760 50  0000 C CNN
-F 2 "" H 9800 1760 60  0000 C CNN
-F 3 "" H 9800 1760 60  0000 C CNN
-	1    9800 1760
+P 9800 1750
+F 0 "P7" H 9800 1850 50  0000 C CNN
+F 1 "CONN_01X01" V 9900 1750 50  0000 C CNN
+F 2 "" H 9800 1750 60  0000 C CNN
+F 3 "" H 9800 1750 60  0000 C CNN
+	1    9800 1750
 	0    1    1    0
 $EndComp
+Wire Wire Line
+	4850 4950 5750 4950
+Connection ~ 4850 4550
+$Comp
+L CONN_01X07 P8
+U 1 1 55813FF5
+P 2650 2150
+F 0 "P8" H 2650 2550 50  0000 C CNN
+F 1 "CONN_01X07" V 2750 2150 50  0000 C CNN
+F 2 "" H 2650 2150 60  0000 C CNN
+F 3 "" H 2650 2150 60  0000 C CNN
+	1    2650 2150
+	1    0    0    -1
+$EndComp
+$Comp
+L GND #PWR018
+U 1 1 558140A3
+P 1700 1950
+F 0 "#PWR018" H 1700 1700 60  0001 C CNN
+F 1 "GND" H 1700 1800 60  0000 C CNN
+F 2 "" H 1700 1950 60  0000 C CNN
+F 3 "" H 1700 1950 60  0000 C CNN
+	1    1700 1950
+	1    0    0    -1
+$EndComp
+Wire Wire Line
+	2450 1850 1700 1850
+Wire Wire Line
+	1700 1850 1700 1950
+$Comp
+L +5V #PWR019
+U 1 1 5581417D
+P 2150 2050
+F 0 "#PWR019" H 2150 1900 60  0001 C CNN
+F 1 "+5V" V 2150 2250 60  0000 C CNN
+F 2 "" H 2150 2050 60  0000 C CNN
+F 3 "" H 2150 2050 60  0000 C CNN
+	1    2150 2050
+	0    -1   -1   0
+$EndComp
+Wire Wire Line
+	2150 2050 2450 2050
+Text Label 2450 2150 2    60   ~ 0
+RX
+Text Label 2450 2250 2    60   ~ 0
+TX
+Text Label 2450 2450 2    60   ~ 0
+DTR
+NoConn ~ 2450 2350
+NoConn ~ 2450 1950
+NoConn ~ 9800 1550
+NoConn ~ 9200 1550
+NoConn ~ 8700 1550
+NoConn ~ 8100 1550
+Connection ~ 5750 4550
 $EndSCHEMATC

Commit message: ADDED NEW FILES
Parts:
- removed P8: CONN_01X07, symbol CONN_01X07
- added P1: CONN_01X07, symbol CONN_01X07
Connections:
- net +5V: now also P1.3 (P3)
- net GND: now also P1.1 (P1)
- net RX: now also P1.4 (P4)
- net TX: now also P1.5 (P5)
- net DTR renamed RESET
- net RESET: now also P1.7 (P7)
Changed lines of the file:
@@
 	1    0    0    -1
 $EndComp
-Wire Wire Line
-	3150 3900 3350 3900
-Wire Wire Line
-	3650 4100 3650 4150
-Wire Wire Line
-	3650 3500 3650 3700
-Wire Wire Line
-	3650 3600 3700 3600
-Connection ~ 3650 3600
-Wire Wire Line
-	4200 3600 4300 3600
-Wire Wire Line
-	4200 3700 4200 3600
-Connection ~ 4200 3600
-Wire Wire Line
-	4600 3800 4600 4150
-Wire Wire Line
-	2550 4350 2550 3900
-Wire Wire Line
-	4200 4150 4200 4100
-Wire Wire Line
-	8430 3210 8680 3210
-Wire Wire Line
-	8530 3210 8530 3260
-Wire Wire Line
-	7380 3210 7630 3210
-Wire Wire Line
-	7530 3210 7530 3260
-Wire Wire Line
-	8030 3510 8030 3660
-Connection ~ 8530 3210
-Connection ~ 7530 3210
-Wire Wire Line
-	5050 2200 5050 2700
-Wire Wire Line
-	5150 2200 5150 2700
-Wire Wire Line
-	5250 2200 5250 2700
-Wire Wire Line
-	5350 2200 5350 2700
-Wire Wire Line
-	5450 2200 5450 2700
-Wire Wire Line
-	5550 2200 5550 2700
-Wire Wire Line
-	5650 2200 5650 2700
-Connection ~ 3200 3900
-Connection ~ 5450 2600
-Wire Wire Line
-	3200 3900 3200 4350
-Wire Wire Line
-	3200 4350 5050 4350
-Connection ~ 5050 4350
-Wire Wire Line
-	5450 2600 4600 2600
-Wire Wire Line
-	4600 2600 4600 3400
-Wire Wire Line
-	3050 4150 3200 4150
-Connection ~ 3200 4150
-Wire Wire Line
-	2650 4150 2550 4150
-Connection ~ 2550 4150
-Wire Wire Line
-	5050 4150 5050 4550
-Wire Wire Line
-	5150 4150 5150 4550
-Wire Wire Line
-	5250 4150 5250 4550
-Wire Wire Line
-	5350 4150 5350 4550
-Wire Wire Line
-	5450 4150 5450 4550
-Wire Wire Line
-	5550 4150 5550 4550
-Wire Wire Line
-	5650 4150 5650 4550
-Wire Wire Line
-	5750 4150 5750 4950
-Wire Wire Line
-	4740 4020 4740 4190
-Wire Wire Line
-	4740 4190 5250 4190
-Connection ~ 5250 4190
-Wire Wire Line
-	5850 4550 5850 4140
-Wire Wire Line
-	5850 4140 6400 4140
-Wire Wire Line
-	6400 4140 6400 3650
-Wire Wire Line
-	6400 3550 6540 3550
-Wire Wire Line
-	6540 3550 6540 4250
-Wire Wire Line
-	6540 4250 5950 4250
-Wire Wire Line
-	5950 4250 5950 4550
-Wire Wire Line
-	6050 4550 6050 4310
-Wire Wire Line
-	6050 4310 6650 4310
-Wire Wire Line
-	6650 4310 6650 3450
-Wire Wire Line
-	6650 3450 6400 3450
-Wire Wire Line
-	4950 4550 4950 4470
-Wire Wire Line
-	4650 4440 4850 4440
-Wire Wire Line
-	4850 4440 4850 4950
-Wire Wire Line
-	4950 2200 4950 2390
-Wire Wire Line
-	4850 2390 4850 2200
-Wire Wire Line
-	4230 2540 5650 2540
-Connection ~ 5650 2540
-Wire Wire Line
-	5750 2700 6040 2700
-Wire Wire Line
-	6040 2700 6040 2730
-Wire Wire Line
-	4230 2010 4230 2040
 $Bitmap
 Pos 9700 5600
@@
 79 E3 73 01 AA 0D CF 9F 3C 98 C5 F6 CF AC 04 72 85 62 D7 80 77 B1 8B CB 18 6F AC E9 6A 17 BB B8
 C2 B0 6B C0 BB D8 C5 65 8C 5D 03 DE C5 2E 2E 63 EC 1A F0 2E 76 71 19 63 D7 80 77 B1 8B CB 18 BB
-06 BC 8B 5D 5C C6 F8 FF 01 52 B3 1C 8C A4 9D 25 1B 00 00 00 00 49 45 4E 44 AE 42 60 82 DA
+06 BC 8B 5D 5C C6 F8 FF 01 52 B3 1C 8C A4 9D 25 1B 00 00 00 00 49 45 4E 44 AE 42 60 82 F5
 EndData
 $EndBitmap
@@
 Text Label 5150 2700 1    60   ~ 0
 RX
-Text Label 4350 4350 0    60   ~ 0
-DTR
 $Comp
 L CONN_01X13 P2
@@
 	0    -1   1    0
 $EndComp
-Wire Wire Line
-	6050 2200 6050 2330
-Wire Wire Line
-	6050 2330 6580 2330
-Wire Wire Line
-	6610 2430 5950 2430
-Wire Wire Line
-	5950 2430 5950 2200
-Wire Wire Line
-	6620 2540 5850 2540
-Wire Wire Line
-	5850 2540 5850 2200
-Wire Wire Line
-	5750 2200 5750 2700
 $Comp
 L CONN_01X01 P4
@@
 	0    1    1    0
 $EndComp
-Wire Wire Line
-	4850 4950 5750 4950
-Connection ~ 4850 4550
 $Comp
-L CONN_01X07 P8
-U 1 1 55813FF5
-P 2650 2150
-F 0 "P8" H 2650 2550 50  0000 C CNN
-F 1 "CONN_01X07" V 2750 2150 50  0000 C CNN
-F 2 "" H 2650 2150 60  0000 C CNN
-F 3 "" H 2650 2150 60  0000 C CNN
-	1    2650 2150
-	1    0    0    -1
+L CONN_01X07 P1
+U 1 1 55A347C2
+P 3300 1350
+F 0 "P1" H 3300 1750 50  0000 C CNN
+F 1 "CONN_01X07" V 3400 1350 50  0000 C CNN
+F 2 "" H 3300 1350 60  0000 C CNN
+F 3 "" H 3300 1350 60  0000 C CNN
+	1    3300 1350
+	-1   0    0    -1
 $EndComp
 $Comp
 L GND #PWR018
-U 1 1 558140A3
-P 1700 1950
-F 0 "#PWR018" H 1700 1700 60  0001 C CNN
-F 1 "GND" H 1700 1800 60  0000 C CNN
-F 2 "" H 1700 1950 60  0000 C CNN
-F 3 "" H 1700 1950 60  0000 C CNN
-	1    1700 1950
+U 1 1 55A3481E
+P 3950 1100
+F 0 "#PWR018" H 3950 850 60  0001 C CNN
+F 1 "GND" H 3950 950 60  0000 C CNN
+F 2 "" H 3950 1100 60  0000 C CNN
+F 3 "" H 3950 1100 60  0000 C CNN
+	1    3950 1100
 	1    0    0    -1
 $EndComp
 Wire Wire Line
-	2450 1850 1700 1850
-Wire Wire Line
-	1700 1850 1700 1950
+	3150 3900 3350 3900
+Wire Wire Line
+	3650 4100 3650 4150
+Wire Wire Line
+	3650 3500 3650 3700
+Wire Wire Line
+	3650 3600 3700 3600
+Connection ~ 3650 3600
+Wire Wire Line
+	4200 3600 4300 3600
+Wire Wire Line
+	4200 3700 4200 3600
+Connection ~ 4200 3600
+Wire Wire Line
+	4600 3800 4600 4150
+Wire Wire Line
+	2550 4350 2550 3900
+Wire Wire Line
+	4200 4150 4200 4100
+Wire Wire Line
+	8430 3210 8680 3210
+Wire Wire Line
+	8530 3210 8530 3260
+Wire Wire Line
+	7380 3210 7630 3210
+Wire Wire Line
+	7530 3210 7530 3260
+Wire Wire Line
+	8030 3510 8030 3660
+Connection ~ 8530 3210
+Connection ~ 7530 3210
+Wire Wire Line
+	5050 2200 5050 2700
+Wire Wire Line
+	5150 2200 5150 2700
+Wire Wire Line
+	5250 2200 5250 2700
+Wire Wire Line
+	5350 2200 5350 2700
+Wire Wire Line
+	5450 2200 5450 2700
+Wire Wire Line
+	5550 2200 5550 2700
+Wire Wire Line
+	5650 2200 5650 2700
+Connection ~ 3200 3900
+Connection ~ 5450 2600
+Wire Wire Line
+	3200 3900 3200 4350
+Wire Wire Line
+	3200 4350 5050 4350
+Connection ~ 5050 4350
+Wire Wire Line
+	5450 2600 4600 2600
+Wire Wire Line
+	4600 2600 4600 3400
+Wire Wire Line
+	3050 4150 3200 4150
+Connection ~ 3200 4150
+Wire Wire Line
+	2650 4150 2550 4150
+Connection ~ 2550 4150
+Wire Wire Line
+	5050 4150 5050 4550
+Wire Wire Line
+	5150 4150 5150 4550
+Wire Wire Line
+	5250 4150 5250 4550
+Wire Wire Line
+	5350 4150 5350 4550
+Wire Wire Line
+	5450 4150 5450 4550
+Wire Wire Line
+	5550 4150 5550 4550
+Wire Wire Line
+	5650 4150 5650 4550
+Wire Wire Line
+	5750 4150 5750 4550
+Wire Wire Line
+	4740 4020 4740 4190
+Wire Wire Line
+	4740 4190 5250 4190
+Connection ~ 5250 4190
+Wire Wire Line
+	5850 4550 5850 4140
+Wire Wire Line
+	5850 4140 6400 4140
+Wire Wire Line
+	6400 4140 6400 3650
+Wire Wire Line
+	6400 3550 6540 3550
+Wire Wire Line
+	6540 3550 6540 4250
+Wire Wire Line
+	6540 4250 5950 4250
+Wire Wire Line
+	5950 4250 5950 4550
+Wire Wire Line
+	6050 4550 6050 4310
+Wire Wire Line
+	6050 4310 6650 4310
+Wire Wire Line
+	6650 4310 6650 3450
+Wire Wire Line
+	6650 3450 6400 3450
+Wire Wire Line
+	4950 4550 4950 4470
+Wire Wire Line
+	4650 4440 4850 4440
+Wire Wire Line
+	4850 4440 4850 4910
+Wire Wire Line
+	4950 2200 4950 2390
+Wire Wire Line
+	4850 2390 4850 2200
+Wire Wire Line
+	4230 2540 5650 2540
+Connection ~ 5650 2540
+Wire Wire Line
+	5750 2700 6040 2700
+Wire Wire Line
+	6040 2700 6040 2730
+Wire Wire Line
+	4230 2010 4230 2040
+Wire Wire Line
+	6050 2200 6050 2330
+Wire Wire Line
+	6050 2330 6580 2330
+Wire Wire Line
+	6610 2430 5950 2430
+Wire Wire Line
+	5950 2430 5950 2200
+Wire Wire Line
+	6620 2540 5850 2540
+Wire Wire Line
+	5850 2540 5850 2200
+Wire Wire Line
+	5750 2200 5750 2700
+Wire Wire Line
+	4850 4910 5750 4910
+Wire Wire Line
+	5750 4910 5750 4540
+Connection ~ 5750 4540
+Connection ~ 4850 4550
+Wire Wire Line
+	3500 1050 3950 1050
+Wire Wire Line
+	3950 1050 3950 1100
+NoConn ~ 3500 1150
 $Comp
 L +5V #PWR019
-U 1 1 5581417D
-P 2150 2050
-F 0 "#PWR019" H 2150 1900 60  0001 C CNN
-F 1 "+5V" V 2150 2250 60  0000 C CNN
-F 2 "" H 2150 2050 60  0000 C CNN
-F 3 "" H 2150 2050 60  0000 C CNN
-	1    2150 2050
-	0    -1   -1   0
+U 1 1 55A34ABF
+P 3800 1250
+F 0 "#PWR019" H 3800 1100 60  0001 C CNN
+F 1 "+5V" H 3930 1310 60  0000 C CNN
+F 2 "" H 3800 1250 60  0000 C CNN
+F 3 "" H 3800 1250 60  0000 C CNN
+	1    3800 1250
+	-1   0    0    1
 $EndComp
 Wire Wire Line
-	2150 2050 2450 2050
-Text Label 2450 2150 2    60   ~ 0
+	3500 1250 3800 1250
+Text Label 3500 1350 0    60   ~ 0
 RX
-Text Label 2450 2250 2    60   ~ 0
+Text Label 3500 1450 0    60   ~ 0
 TX
-Text Label 2450 2450 2    60   ~ 0
-DTR
-NoConn ~ 2450 2350
-NoConn ~ 2450 1950
+NoConn ~ 3500 1550
+Text Label 3500 1650 0    40   ~ 0
+RESET
+NoConn ~ 8100 1550
+NoConn ~ 8700 1550
+NoConn ~ 9200 1550
 NoConn ~ 9800 1550
-NoConn ~ 9200 1550
-NoConn ~ 8700 1550
-NoConn ~ 8100 1550
-Connection ~ 5750 4550
 $EndSCHEMATC
