File: ESP12E BOB_1.kicad_pcb (KiCad board)
At the start: 2 copper layers, 26.5 x 43.5 mm, 21 parts, among them M1 ESP-12E, P1 CONN_01X07, P2 CONN_01X13, P3 CONN_01X13, P4 CONN_01X01, P5 CONN_01X01, P6 CONN_01X01, P7 CONN_01X01, Q1 BSS138, Q2 BSS138, SW1 SW_PUSH, U1 1117-3.3

Commit message: added corrected files
Other:
- outline, holes or cut-outs redrawn
- board text added: "GND"
Changed lines of the file:
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@@
     (links 55)
     (no_connects 0)
-    (area 112.399999 40.899999 139.100001 84.600001)
+    (area 109.091667 40.768 142.368334 84.600001)
     (thickness 1.6)
-    (drawings 43)
+    (drawings 47)
     (tracks 244)
     (zones 0)
@@
   )
   (setup
-    (last_trace_width 0.635)
+    (last_trace_width 0.35)
     (user_trace_width 0.3048)
     (user_trace_width 0.381)
@@
       (xy 7 -5.15)) (layer B.SilkS) (width 0.01))
   )
-  (gr_line (start 112.5 43.5) (end 112.5 84.5) (angle 90) (layer Edge.Cuts) (width 0.2))
+  (gr_line (start 115 84.5) (end 136.5 84.5) (angle 90) (layer Edge.Cuts) (width 0.2))
+  (gr_line (start 112.5 44) (end 112.5 82) (angle 90) (layer Edge.Cuts) (width 0.2))
+  (gr_line (start 139 82) (end 139 44.5) (angle 90) (layer Edge.Cuts) (width 0.2))
+  (gr_line (start 112.5 41) (end 115.5 41) (angle 90) (layer Edge.Cuts) (width 0.2))
+  (gr_line (start 112.5 44) (end 112.5 41) (angle 90) (layer Edge.Cuts) (width 0.2))
+  (gr_line (start 139 41) (end 136 41) (angle 90) (layer Edge.Cuts) (width 0.2))
+  (gr_line (start 139 44.5) (end 139 41) (angle 90) (layer Edge.Cuts) (width 0.2))
+  (gr_arc (start 136.5 82) (end 139 82) (angle 90) (layer Edge.Cuts) (width 0.2))
+  (gr_arc (start 115 82) (end 115 84.5) (angle 90) (layer Edge.Cuts) (width 0.2))
   (gr_line (start 136.5 41) (end 115 41) (angle 90) (layer Edge.Cuts) (width 0.2))
-  (gr_line (start 139 84.5) (end 139 43.5) (angle 90) (layer Edge.Cuts) (width 0.2))
-  (gr_arc (start 136.5 43.5) (end 136.5 41) (angle 90) (layer Edge.Cuts) (width 0.2))
-  (gr_arc (start 115 43.5) (end 112.5 43.5) (angle 90) (layer Edge.Cuts) (width 0.2))
-  (gr_line (start 139 84.5) (end 112.5 84.5) (angle 90) (layer Edge.Cuts) (width 0.2))
   (gr_text DTR (at 117.856 45.339) (layer F.SilkS)
     (effects (font (size 0.889 0.889) (thickness 0.22225)))
   )
-  (gr_text NC (at 130.683 45.339) (layer F.SilkS)
+  (gr_text NC (at 130.556 45.339) (layer F.SilkS)
     (effects (font (size 0.889 0.889) (thickness 0.22225)))
   )
@@
     (effects (font (size 0.889 0.889) (thickness 0.22225)))
   )
-  (gr_text G (at 132.969 45.339) (layer F.SilkS)
+  (gr_text "GND\n" (at 133.096 45.339) (layer F.SilkS)
     (effects (font (size 0.889 0.889) (thickness 0.22225)))
   )
@@
     (effects (font (size 1 1) (thickness 0.2)) (justify mirror))
   )
-  (segment (start 133.096 43.053) (end 133.096 49.657) (width 0.635) (layer F.Cu) (net 1) (status 400000))
-  (segment (start 134.239 50.8) (end 137.16 50.8) (width 0.635) (layer F.Cu) (net 1) (status 800000))
+  (segment (start 133.096 43.053) (end 133.096 49.657) (width 0.635) (layer F.Cu) (net 1))
+  (segment (start 134.239 50.8) (end 137.16 50.8) (width 0.635) (layer F.Cu) (net 1))
   (segment (start 133.096 49.657) (end 134.239 50.8) (width 0.635) (layer F.Cu) (net 1))
   (segment (start 128.524 78.232) (end 132.334 78.232) (width 0.762) (layer B.Cu) (net 1))
@@
   (segment (start 128.016 66.04) (end 130.386 63.67) (width 0.35) (layer B.Cu) (net 2))
   (segment (start 130.386 63.67) (end 130.386 61.468) (width 0.35) (layer B.Cu) (net 2))
-  (segment (start 128.016 43.053) (end 128.016 44.577) (width 0.635) (layer B.Cu) (net 3) (status 400000))
+  (segment (start 128.016 43.053) (end 128.016 44.577) (width 0.635) (layer B.Cu) (net 3))
   (segment (start 128.016 44.577) (end 126.619 45.974) (width 0.635) (layer B.Cu) (net 3))
   (segment (start 137.16 48.26) (end 132.61086 48.26) (width 0.635) (layer B.Cu) (net 3))
@@
   (segment (start 135.096 59.468) (end 136.144 58.42) (width 0.508) (layer F.Cu) (net 21))
   (segment (start 136.144 58.42) (end 137.16 58.42) (width 0.508) (layer F.Cu) (net 21))
-  (segment (start 122.936 43.053) (end 122.936 45.212) (width 0.508) (layer F.Cu) (net 22) (status 400000))
+  (segment (start 122.936 43.053) (end 122.936 45.212) (width 0.508) (layer F.Cu) (net 22))
   (segment (start 126.492 48.768) (end 126.492 54.61) (width 0.508) (layer F.Cu) (net 22))
   (segment (start 122.936 45.212) (end 126.492 48.768) (width 0.508) (layer F.Cu) (net 22))
@@
   (segment (start 134.62 53.34) (end 137.16 53.34) (width 0.35) (layer F.Cu) (net 22))
   (segment (start 133.73 54.23) (end 134.62 53.34) (width 0.35) (layer F.Cu) (net 22))
-  (segment (start 125.476 43.053) (end 125.476 44.831) (width 0.508) (layer F.Cu) (net 23) (status 400000))
+  (segment (start 125.476 43.053) (end 125.476 44.831) (width 0.508) (layer F.Cu) (net 23))
   (segment (start 127.572 57.468) (end 130.492 57.468) (width 0.508) (layer F.Cu) (net 23))
   (segment (start 124.968 54.864) (end 127.572 57.468) (width 0.508) (layer F.Cu) (net 23))
@@
   (segment (start 124.46 60.96) (end 124.46 57.404) (width 0.635) (layer B.Cu) (net 24))
   (segment (start 124.968 61.468) (end 124.46 60.96) (width 0.635) (layer B.Cu) (net 24))
-  (segment (start 118.73 55.468) (end 118.73 53.98) (width 0.635) (layer F.Cu) (net 29) (status 400000))
-  (segment (start 118.09 53.34) (end 114.3 53.34) (width 0.635) (layer F.Cu) (net 29) (status 800000))
+  (segment (start 118.73 55.468) (end 118.73 53.98) (width 0.635) (layer F.Cu) (net 29))
+  (segment (start 118.09 53.34) (end 114.3 53.34) (width 0.635) (layer F.Cu) (net 29))
   (segment (start 118.73 53.98) (end 118.09 53.34) (width 0.635) (layer F.Cu) (net 29))
-  (segment (start 117.856 43.053) (end 117.856 52.324) (width 0.635) (layer F.Cu) (net 29) (status 400000))
+  (segment (start 117.856 43.053) (end 117.856 52.324) (width 0.635) (layer F.Cu) (net 29))
   (segment (start 117.856 52.324) (end 116.84 53.34) (width 0.635) (layer F.Cu) (net 29))
   (segment (start 123.444 78.232) (end 123.444 71.12) (width 0.762) (layer B.Cu) (net 29))
@@
   (segment (start 116.586 53.848) (end 116.078 53.34) (width 0.635) (layer B.Cu) (net 29))
   (segment (start 116.078 53.34) (end 114.3 53.34) (width 0.635) (layer B.Cu) (net 29))
-  (zone (net 4) (net_name +3V3) (layer F.Cu) (hatch edge 0.508)
+  (zone (net 1) (net_name GND) (layer B.Cu) (hatch edge 0.508)
     (connect_pads (clearance 0.508))
     (min_thickness 0.254)
@@
     (polygon
       (pts
-        (xy 139 43.75) (xy 139 84.5) (xy 112.5 84.5) (xy 112.5 43.5) (xy 112.75 42.5)
-        (xy 113 42) (xy 113.5 41.5) (xy 114 41.25) (xy 114.75 41) (xy 136.5 41)
-        (xy 137.5 41.25) (xy 138.25 41.75) (xy 138.5 42) (xy 138.75 42.5) (xy 139 43.5)
-        (xy 139 43.75)
+        (xy 139 82) (xy 138.5 83.5) (xy 137 84.5) (xy 115 84.5) (xy 113.5 84)
+        (xy 112.5 82.5) (xy 112.5 41) (xy 139 41)
       )
     )
   )
-  (zone (net 1) (net_name GND) (layer B.Cu) (hatch edge 0.508)
+  (zone (net 4) (net_name +3V3) (layer F.Cu) (hatch edge 0.508)
     (connect_pads (clearance 0.508))
     (min_thickness 0.254)
@@
     (polygon
       (pts
-        (xy 139 43.5) (xy 139 84.5) (xy 112.5 84.5) (xy 112.5 43.75) (xy 112.5 43.25)
-        (xy 112.75 42.5) (xy 113.25 41.75) (xy 113.75 41.25) (xy 115 41) (xy 136.75 41)
-        (xy 137.5 41.25) (xy 138.25 41.75) (xy 138.75 42.5) (xy 139 43.25) (xy 139 43.5)
+        (xy 139 82) (xy 138.5 83.5) (xy 137 84.5) (xy 115 84.5) (xy 113.5 84)
+        (xy 112.5 82.5) (xy 112.5 41) (xy 139 41)
       )
     )
